Commit message: dev : data collection

File: src/flintrobot_description/urdf/flintrobot_base_no1.urdf (robot description, URDF)
Before this commit: robot flintrobot, 55 links, 54 joints
Links:
- link body_link: geometry collision cylinder length=0.95 radius=0.15; visual cylinder length=0.95 radius=0.15
